Commit message: proper Link0 Link1

File: body.urdf (robot description, URDF)
Before this commit: robot robot, 2 links, 1 joints
Joints:
- joint Link0_Link1: origin xyz=0 0 0 rpy=0 0 0 -> xyz=0 0 1 rpy=0 0 0

Commit message: Link 0 Link 1 Link 2

File: body.urdf (robot description, URDF)
Before this commit: robot robot, 2 links, 1 joints
Links:
- added link Link2, mass 1; collision box size=1 1 1; visual box size=1 1 1
Joints:
- added joint Link1_Link2: type revolute, parent Link1, child Link2, origin xyz=0 0 1 rpy=0 0 0, axis 0 1 0, limit lower=-3.14159 upper=3.14159 effort=0.0 velocity=0.0

Commit message: link 0,1, 2, 3, 4

File: body.urdf (robot description, URDF)
Before this commit: robot robot, 3 links, 2 joints
Links:
- added link Link3, mass 1; collision box size=1 1 1; visual box size=1 1 1
- added link Link4, mass 1; collision box size=1 1 1; visual box size=1 1 1
Joints:
- added joint Link2_Link3: type revolute, parent Link2, child Link3, origin xyz=0 0 1 rpy=0 0 0, axis 0 1 0, limit lower=-3.14159 upper=3.14159 effort=0.0 velocity=0.0
- added joint Link3_Link4: type revolute, parent Link3, child Link4, origin xyz=0 0.5 0.5 rpy=0 0 0, axis 0 1 0, limit lower=-3.14159 upper=3.14159 effort=0.0 velocity=0.0

Commit message: fixed part e

File: body.urdf (robot description, URDF)
Before this commit: robot robot, 5 links, 4 joints
Links:
- removed link Link3
- removed link Link4
Joints:
- removed joint Link1_Link2
- removed joint Link2_Link3
- removed joint Link3_Link4
- added joint Link0_Link2: type revolute, parent Link0, child Link2, origin xyz=1 0 1 rpy=0 0 0, axis 0 1 0, limit lower=-3.14159 upper=3.14159 effort=0.0 velocity=0.0
- joint Link0_Link1: origin xyz=0 0 1 rpy=0 0 0 -> xyz=2 0 1 rpy=0 0 0

Commit message: sensor setup

File: body.urdf (robot description, URDF)
Before this commit: robot robot, 5 links, 4 joints
Links:
- removed link Link0
- removed link Link1
- removed link Link2
- removed link Link3
- removed link Link4
- added link BackLeg, mass 1; collision box size=1 1 1; visual box size=1 1 1
- added link FrontLeg, mass 1; collision box size=1 1 1; visual box size=1 1 1
- added link Torso, mass 1; collision box size=1 1 1; visual box size=1 1 1
Joints:
- removed joint Link0_Link1
- removed joint Link1_Link2
- removed joint Link2_Link3
- removed joint Link3_Link4
- added joint Torso_BackLeg: type revolute, parent Torso, child BackLeg, origin xyz=2 0 1 rpy=0 0 0, axis 0 1 0, limit lower=-3.14159 upper=3.14159 effort=0.0 velocity=0.0
- added joint Torso_FrontLeg: type revolute, parent Torso, child FrontLeg, origin xyz=1 0 1 rpy=0 0 0, axis 0 1 0, limit lower=-3.14159 upper=3.14159 effort=0.0 velocity=0.0
